Commit message: added Lidar and Camera Sensors.

File: dd_gazebo_ws/dd_gazebo/src/description/drone_description.urdf (robot description, URDF)
Before this commit: robot drone, 2 links, 1 joints
Links:
- added link base_footprint
- added link camera_depth_frame
- added link camera_link, mass 0.035; collision box size=0.015 0.130 0.022; visual box size=0.015 0.130 0.022
- added link lidar_link, mass 0.125; collision cylinder length=0.055 radius=0.0508; visual cylinder length=0.045 radius=0.0408
Joints:
- added joint base_joint: type fixed, parent base_link, child base_footprint, origin xyz=0.0 0.0 ${-(base_link_height)} rpy=0 0 0
- added joint camera_depth_joint: type fixed, parent camera_link, child camera_depth_frame, origin xyz=0 0 0 rpy=${-pi/2} 0 ${-pi/2}
- added joint camera_joint: type fixed, parent base_link, child camera_link, origin xyz=0.26 0 0.045 rpy=0 0 0
- added joint lidar_joint: type fixed, parent base_link, child lidar_link, origin xyz=0 0 0.08 rpy=0 0 0
- joint imu_joint: origin xyz=0 0 0.01 -> xyz=0 0 0.008
