Commit message: Added 3d lidar sensor and depth camera to model velodyne and Zed2i sensors.

File: dd_gazebo_ws/src/drone_nav/description/drone_model.urdf (robot description, URDF)
Before this commit: robot typhoon_h480, 16 links, 15 joints
Links:
- added link depth_camera_optical_link
Joints:
- added joint depth_camera_optical_joint: type fixed, parent camera_link, child depth_camera_optical_link, origin xyz=0 0 0 rpy=-1.57079632679 0 -1.57079632679, axis 0 0 0
